File: circuit/basic_f051r8/basic_f051r8.kicad_sch (KiCad schematic)
At the start: 1 part

Commit message: Schematic
Parts:
- added C1, C3, C5: 100uF, symbol Device:C_Polarized
- added C2, C4, C6, C7: 100nF, symbol Device:C
- added D1, D2, D4: LED, symbol Device:LED
- added D3: D, symbol Device:D
- added J1: Conn_01x04_Male, symbol Connector:Conn_01x04_Male
- added J2: Conn_01x03_Male, symbol Connector:Conn_01x03_Male
- added J3: USB_B, symbol Connector:USB_B
- added Q1: 2N3904, Package_TO_SOT_THT:TO-92_Inline, symbol Transistor_BJT:2N3904
- added R1: 0, symbol Device:R
- added R10: 10K, symbol Device:R
- added R11, R12, R6: 1k, symbol Device:R
- added R2, R3, R7: 10k, symbol Device:R
- added R4, R5: 220, symbol Device:R
- added R8, R9: 330, symbol Device:R
- added SW1, SW2: SW_Push, symbol Switch:SW_Push
- added U2: AMS1117-5.0, Package_TO_SOT_SMD:SOT-223-3_TabPin2, symbol Regulator_Linear:AMS1117-5.0
- added U3: H11L1, symbol Isolator:H11L1
- added U4: FT232RL, Package_SO:SSOP-28_5.3x10.2mm_P0.65mm, symbol Interface_USB:FT232RL
- gave numbers to parts that had none: 1
Connections:
- net IN_CRANK: now also R10.2, U3.4
- net IN_TPS: now also C7.2, R11.2, R12.2
- net LED_NOPULSE: now also D1.1 (K)
- net RX: now also U4.1 (TXD)
- net TX: now also U4.5 (RXD)
- net VDD: now reaches U1.1 (VBAT)
- net VDD: now also U1.13 (VDDA), U1.32 (VDD), U1.64 (VDD), C1.1, C2.1, J1.1 (Pin_1), R10.1, R3.1, R4.1, R5.1, R8.1, R9.1, SW1.2, U3.6, U4.17 (3V3OUT), U4.4 (VCCIO)
- net GND: now reaches U1.12 (VSSA)
- net GND: now also U1.31 (VSS), U1.63 (VSS), C1.2, C2.2, C4.1, C5.1, C6.1, C7.1, D2.1 (K), D3.2 (A), J1.3 (Pin_3), J2.3 (Pin_3), J3.4 (GND), J3.5 (Shield), Q1.1 (E), R1.2, R12.1, R2.2, R7.2, SW2.2, U2.1 (GND), U3.5, U4.18 (GND), U4.21 (GND), U4.25 (AGND), U4.26 (TEST), U4.7 (GND)
- net at U1.28 (PB2): now also R1.1
- net SWD_IO: now reaches U1.46 (PA13)
- net SWD_IO: now also J1.4 (Pin_4)
- net SWD_CLK: now reaches U1.49 (PA14)
- net SWD_CLK: now also J1.2 (Pin_2)
- net BOOT0: now reaches U1.60 (BOOT0)
- net BOOT0: now also R2.1, SW1.1
- net NRST: now reaches U1.7 (NRST)
- net NRST: now also R3.2, SW2.1
- new net: D4.1 (K), Q1.3 (C), U3.2
- new net: D4.2 (A), R8.2
- new net: D1.2 (A), R4.2
- new net: D2.2 (A), R5.2
- new net: C6.2, Q1.2 (B), R6.2, R7.1
- new net: J3.2 (D-), U4.16 (USBD-)
- new net: J3.3 (D+), U4.15 (USBD+)
- new net: J2.2 (Pin_2), R11.1
- new net: R9.2, U3.1
- new net +12V: C3.1, U2.3 (VI)
- new net CRANK_PORT: R6.1
- new net GNDPWR: C3.2, D3.1 (K)
- new net VCC: C4.2, C5.2, J2.1 (Pin_1), U2.2 (VO), U4.20 (VCC)
- no-connect marks 0 -> 58
Other:
- note added: "5V LDO"
- note added: "MAIN CHIP"
- note added: "PULSER INPUT"
- note added: "TPS INPUT"
- note added: "USB SERIAL"
- moved on the sheet: U1

Commit message: Schematic Done
Parts:
- added H1, H2, H3, H4: MountingHole, symbol Mechanical:MountingHole
- added J4, J5, J6, J7: Conn_01x02_Male, symbol Connector:Conn_01x02_Male
- added Q2, Q3, Q4, Q5: IRF540N, Package_TO_SOT_THT:TO-220-3_Vertical, symbol Transistor_FET:IRF540N
- added R13, R16, R19, R22: 220, symbol Device:R
- added R14, R15, R17, R18, R20, R21, R23, R24: 10k, symbol Device:R
- added U5, U6, U7, U8: 4N35, Package_DIP:DIP-6_W7.62mm, symbol Isolator:4N35
Connections:
- net +12V: now also J4.1 (Pin_1), R14.1, R15.1, R17.1, R18.1, R20.1, R21.1, R23.1, R24.1
- net CRANK_PORT: now also J6.1 (Pin_1)
- net GND: now also J6.2 (Pin_2)
- net GNDPWR: now also J4.2 (Pin_2), Q2.3 (S), Q3.3 (S), Q4.3 (S), Q5.3 (S), U5.4, U6.4, U7.4, U8.4
- net OUT_IGNA: now also U7.2
- net OUT_IGNB: now also U8.2
- net OUT_INJA: now also U5.2
- net OUT_INJB: now also U6.2
- net VDD: now also R13.1, R16.1, R19.1, R22.1
- new net: Q3.1 (G), R17.2, U6.5
- new net: Q2.1 (G), R14.2, U5.5
- new net: Q4.1 (G), R20.2, U7.5
- new net: R22.2, U8.1
- new net: R19.2, U7.1
- new net: R16.2, U6.1
- new net: R13.2, U5.1
- new net: Q5.1 (G), R23.2, U8.5
- new net PORT_IGNA: J5.1 (Pin_1), Q4.2 (D), R21.2
- new net PORT_IGNB: J5.2 (Pin_2), Q5.2 (D), R24.2
- new net PORT_INJA: J7.1 (Pin_1), Q2.2 (D), R15.2
- new net PORT_INJB: J7.2 (Pin_2), Q3.2 (D), R18.2
- no-connect marks 58 -> 62
Other:
- note added: "ENGINE CONTROL"
- note added: "ENGINE PORT"
- note added: "HOLES"
- company: (none) -> Achmadi ST MT
- title: (none) -> Custom Engine Control Unit

Commit message: Footprint Assigment
Parts:
- C1, C2, C3, C4, C5, C6, C7: footprint (none) -> Capacitor_SMD:C_0805_2012Metric_Pad1.18x1.45mm_HandSolder
- D1, D2, D4: footprint (none) -> LED_SMD:LED_0805_2012Metric_Pad1.15x1.40mm_HandSolder
- D3: footprint (none) -> Diode_SMD:D_SMA-SMB_Universal_Handsoldering
- H1, H2, H3, H4: footprint (none) -> MountingHole:MountingHole_2.5mm_Pad
- J1: footprint (none) -> Connector_PinHeader_2.54mm:PinHeader_1x04_P2.54mm_Vertical
- J2: footprint (none) -> TerminalBlock:TerminalBlock_Altech_AK300-3_P5.00mm
- J3: footprint (none) -> Connector_USB:USB_B_Lumberg_2411_02_Horizontal
- J4, J5, J6, J7: footprint (none) -> TerminalBlock:TerminalBlock_Altech_AK300-2_P5.00mm
- R1, R10, R11, R12, R13, R14, R15, R16, R17, R18, R19, R2, R20, R21, R22, R23, R24, R3, R4, R5, R6, R7, R8, R9: footprint (none) -> Resistor_SMD:R_0805_2012Metric_Pad1.20x1.40mm_HandSolder
- SW1, SW2: footprint (none) -> Button_Switch_THT:SW_PUSH_6mm
- U3: footprint (none) -> Package_DIP:DIP-6_W7.62mm

Commit message: PCB Layout (No Route)
Parts:
- C1, C5: footprint Capacitor_SMD:C_0805_2012Metric_Pad1.18x1.45mm_HandSolder -> Capacitor_SMD:C_Elec_4x5.4
- Q2, Q3, Q4, Q5: footprint Package_TO_SOT_THT:TO-220-3_Vertical -> Package_TO_SOT_THT:TO-220-3_Horizontal_TabUp
Changed lines of the file:
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@@
   (no_connect (at 59.69 60.96))
   (no_connect (at 59.69 58.42))
+  (no_connect (at 29.21 68.58))
   (no_connect (at 29.21 60.96))
   (no_connect (at 29.21 63.5))
-  (no_connect (at 29.21 68.58))
   (no_connect (at 29.21 58.42))
   (no_connect (at 29.21 50.8))
@@
     (effects (font (size 2 2) bold) (justify left bottom))
   )
-  (text "USB SERIAL\n" (at 209.55 120.65 0)
+  (text "USB SERIAL\n" (at 201.93 123.19 0)
     (effects (font (size 2 2) bold) (justify left bottom))
   )
@@
       (effects (font (size 1.27 1.27)) (justify left))
     )
-    (property "Footprint" "Capacitor_SMD:C_0805_2012Metric_Pad1.18x1.45mm_HandSolder" (id 2) (at 70.8152 110.49 0)
+    (property "Footprint" "Capacitor_SMD:C_Elec_4x5.4" (id 2) (at 70.8152 110.49 0)
       (effects (font (size 1.27 1.27)) hide)
     )
@@
       (effects (font (size 1.27 1.27)) (justify left))
     )
-    (property "Footprint" "Package_TO_SOT_THT:TO-220-3_Vertical" (id 2) (at 125.73 151.765 0)
+    (property "Footprint" "Package_TO_SOT_THT:TO-220-3_Horizontal_TabUp" (id 2) (at 125.73 151.765 0)
       (effects (font (size 1.27 1.27) italic) (justify left) hide)
     )
@@
       (effects (font (size 1.27 1.27)) (justify left))
     )
-    (property "Footprint" "Capacitor_SMD:C_0805_2012Metric_Pad1.18x1.45mm_HandSolder" (id 2) (at 170.4848 29.21 0)
+    (property "Footprint" "Capacitor_SMD:C_Elec_4x5.4" (id 2) (at 170.4848 29.21 0)
       (effects (font (size 1.27 1.27)) hide)
     )
@@
       (effects (font (size 1.27 1.27)) (justify left))
     )
-    (property "Footprint" "Package_TO_SOT_THT:TO-220-3_Vertical" (id 2) (at 60.96 156.845 0)
+    (property "Footprint" "Package_TO_SOT_THT:TO-220-3_Horizontal_TabUp" (id 2) (at 60.96 156.845 0)
       (effects (font (size 1.27 1.27) italic) (justify left) hide)
     )
@@
       (effects (font (size 1.27 1.27)) (justify left))
     )
-    (property "Footprint" "Package_TO_SOT_THT:TO-220-3_Vertical" (id 2) (at 76.2 184.785 0)
+    (property "Footprint" "Package_TO_SOT_THT:TO-220-3_Horizontal_TabUp" (id 2) (at 76.2 184.785 0)
       (effects (font (size 1.27 1.27) italic) (justify left) hide)
     )
@@
       (effects (font (size 1.27 1.27)) (justify left))
     )
-    (property "Footprint" "Package_TO_SOT_THT:TO-220-3_Vertical" (id 2) (at 138.43 184.785 0)
+    (property "Footprint" "Package_TO_SOT_THT:TO-220-3_Horizontal_TabUp" (id 2) (at 138.43 184.785 0)
       (effects (font (size 1.27 1.27) italic) (justify left) hide)
     )
@@
     )
     (path "/0ad63f58-6d9a-4abb-9e66-60bf54110f75"
-      (reference "C1") (unit 1) (value "100uF") (footprint "Capacitor_SMD:C_0805_2012Metric_Pad1.18x1.45mm_HandSolder")
+      (reference "C1") (unit 1) (value "100uF") (footprint "Capacitor_SMD:C_Elec_4x5.4")
     )
     (path "/7fff78ec-489e-46d1-97a7-74d2ede59843"
@@
     )
     (path "/32a9317a-3560-4758-bb05-c3f3031deca0"
-      (reference "C5") (unit 1) (value "100uF") (footprint "Capacitor_SMD:C_0805_2012Metric_Pad1.18x1.45mm_HandSolder")
+      (reference "C5") (unit 1) (value "100uF") (footprint "Capacitor_SMD:C_Elec_4x5.4")
     )
     (path "/77e9475f-b577-4388-96b7-363fc9dc62b5"
@@
     )
     (path "/8e154746-f067-4634-8a5e-a8202f041c8f"
-      (reference "Q2") (unit 1) (value "IRF540N") (footprint "Package_TO_SOT_THT:TO-220-3_Vertical")
+      (reference "Q2") (unit 1) (value "IRF540N") (footprint "Package_TO_SOT_THT:TO-220-3_Horizontal_TabUp")
     )
     (path "/efa2572f-c7c6-4ccb-9220-5504cf7dcc28"
-      (reference "Q3") (unit 1) (value "IRF540N") (footprint "Package_TO_SOT_THT:TO-220-3_Vertical")
+      (reference "Q3") (unit 1) (value "IRF540N") (footprint "Package_TO_SOT_THT:TO-220-3_Horizontal_TabUp")
     )
     (path "/20581314-518f-4b8d-b3b8-19764e8655b3"
-      (reference "Q4") (unit 1) (value "IRF540N") (footprint "Package_TO_SOT_THT:TO-220-3_Vertical")
+      (reference "Q4") (unit 1) (value "IRF540N") (footprint "Package_TO_SOT_THT:TO-220-3_Horizontal_TabUp")
     )
     (path "/f18470ea-0575-448a-9d8a-dbd68b3f9cac"
-      (reference "Q5") (unit 1) (value "IRF540N") (footprint "Package_TO_SOT_THT:TO-220-3_Vertical")
+      (reference "Q5") (unit 1) (value "IRF540N") (footprint "Package_TO_SOT_THT:TO-220-3_Horizontal_TabUp")
     )
     (path "/3862d9a3-19ea-4fd9-8143-3593b521e976"
